File: xmega.kicad_pcb (KiCad board)
At the start: 2 copper layers, 100 x 100 mm, 98 parts, among them J1 USB, J2 PORTA, J3 PDI, J4 PORTB, J5 PORTC, J6 PORTE, J7 AUX, J8 MCU_CURRENT, J9 RAM_CURRENT, Q1 MMUN2231L, Q2 IRLML6402, SW1 PF0, SW2 PF1, SW3 PF2, SW4 PF3, SW5 RST, U1 ATXMEGA128A1U-AU, U2 SN74AHC573PW, U3 IDT71V256SA, U4 LM3671MF, U5 M24C02-WDW6TP, U6 ADR380, X1 16MHz, X2 32768

Commit message: Finished?
Parts:
- removed C33: 100n, IPC7351-Nominal:CAPC1005X55
- removed the G*** at (92.0, 8.00)
- removed Q2: IRLML6402, smd-semi:SOT-23
- added G***: LOGO, LOGO, B.Cu at (13.2, 13.8)
- added G***: LOGO, LOGO, B.Cu at (86.8, 13.8)
- added G***: LOGO, LOGO, B.Cu at (13.3, 85.1)
- added J10: POWER, conn-fci:CONN-10118194-0001LF-FCI, F.Cu at (88.0, 1.50)
- added R16: 365, IPC7351-Nominal:RESC1005X40, F.Cu at (27.8, 85.0)
- added R17: 3k3, IPC7351-Nominal:RESCAXE80P160X320X70-8, F.Cu at (24.5, 85.0)
- added TP1: GND, manuf:TESTPOINT-KEYSTONE-5018, F.Cu at (35.0, 79.0)
- added U7: TPS2110A, IPC7351-Nominal:SOP65P640X110-8, F.Cu at (23.5, 91.0)
- R13: value 100k -> 365; footprint IPC7351-Nominal:RESCAXE80P160X320X70-8 -> IPC7351-Nominal:RESC1005X40
- moved C32 106.1 mm to (88.0, 7.50), turned to 0 degrees
- moved R13 2.80 mm to (20.8, 88.5), turned to 90 degrees
- moved FID1 1.68 mm to (30.0, 82.8)
Connections:
- C28 pad 1: (no net) -> 3V3RAM
- C28 pad 2: (no net) -> GND
- C32 pad 1: Net-(C32-Pad1) -> GND
- C32 pad 2: /Power/FILT_VBUS -> /Power/ALT_VBUS
- C4 pad 1: (no net) -> 3V3RAM
- C4 pad 2: (no net) -> GND
- J9 pad 1: (no net) -> 3V3RAM
- J9 pad 2: (no net) -> +3.3
- R13 pad 1: GND -> Net-(R13-Pad1)
- R15 pad 1: (no net) -> 3V3RAM
- R15 pad 2: (no net) -> +3.3
Routing:
- net /Power/ALT_VBUS: track 0.00 -> 164.9 mm, vias 0 -> 2
- net GND: track 518.7 -> 540.8 mm, vias 155 -> 174
- net Net-(C32-Pad1): track 12.4 -> 0.00 mm
- net VBUS: track 9.38 -> 14.2 mm
- net +3.3: track 214.9 -> 211.7 mm
- net Net-(R17-Pad5): track 0.00 -> 3.00 mm
- net /Power/FILT_VBUS: track 4.47 -> 1.63 mm
- net Net-(R13-Pad1): track 0.00 -> 2.54 mm
- net Net-(R16-Pad2): track 0.00 -> 2.24 mm
- net /Management/RESET: track 128.0 -> 126.5 mm
- net (no net): track 1.55 -> 0.00 mm, vias 1 -> 0
- net Net-(R17-Pad7): track 0.00 -> 0.80 mm
- net Net-(R17-Pad2): track 0.00 -> 0.80 mm
- added copper zone on F.Cu, net /Power/ALT_VBUS
Other:
- board text added: "AUX POWER"
- board text added: "CC0 1.0 — REV 1 — 2016-03"
- board text added: "Preferred when present"
- board text removed: "CC0 1.0"
- board text removed: "REV 1 — 2016-03"

Commit message: Reannotate
Parts:
- renumbered C22 to C1, C30 to C10, C31 to C11, C32 to C12, C35 to C13, C24 to C14, C25 to C15, C26 to C16, C3 to C17, C6 to C18, C5 to C19, C23 to C2, C4 to C20, C8 to C21, C7 to C22, C28 to C23, C10 to C24, C9 to C25, C34 to C26, C12 to C27, C11 to C28, C13 to C29, C29 to C3, C27 to C30, C1 to C31, C2 to C32, C20 to C33, C21 to C34, C14 to C4, C15 to C5, C16 to C6, C17 to C7, C18 to C8, C19 to C9, DS5 to DS1, DS1 to DS2, DS2 to DS3, DS3 to DS4, DS4 to DS5, J7 to J10, J4 to J3, J5 to J4, J6 to J5, J3 to J6, J10 to J7, L2 to L1, R9 to R10, R23 to R11, R25 to R12, R26 to R13, R24 to R14, R19 to R15, R10 to R16, R11 to R17, R14 to R18, R15 to R19, R16 to R20, R17 to R21, R13 to R22, R12 to R9, SW5 to SW1, SW1 to SW2, SW2 to SW3, SW3 to SW4, SW4 to SW5, TP3 to TP1, TP5 to TP2, TP6 to TP3, TP1 to TP5, U6 to U2, U5 to U3, U2 to U4, U3 to U5, U7 to U6, U4 to U7
Other:
- net class Default: clearance 0.2 -> 0.199
- rule trace_clearance: 0.2 -> 0.199

Commit message: Schematic tidy-ups and add VBUS sense
Parts:
- removed the G*** at (13.2, 13.8)
- removed the G*** at (86.8, 13.8)
- added R23: 3k3, IPC7351-Nominal:RESCAXE80P160X320X70-8, F.Cu at (12.0, 85.8)
- JP1: value JUMPER -> PA0
- JP2: value JUMPER -> PB0
- moved G*** 64.3 mm to (77.6, 85.0)
Connections:
- net /LS_SCL renamed /EEP_SCL
- net /LS_SDA renamed /EEP_SDA
- net /LS_V+ renamed /EEP_V+
- net /PD3 renamed /VR_V+
- net /Power/ALT_VBUS renamed /Power/ALT_VBUS_IN
- net Net-(C10-Pad1) renamed /Management/TOSC2
- net Net-(C11-Pad1) renamed /Management/TOSC1
- net Net-(C8-Pad1) renamed /Management/XTAL1
- net Net-(C9-Pad1) renamed /Management/XTAL2
Routing:
- net Net-(R23-Pad7): track 2.05 -> 51.0 mm, vias 0 -> 2
- net GND: track 540.8 -> 546.1 mm
- net /LD-: track 65.6 -> 67.2 mm
- net /LD+: track 65.8 -> 67.4 mm
- net /E_VBUS: track 10.9 -> 12.4 mm
Other:
- net class Default: clearance 0.199 -> 0.2
- rule trace_clearance: 0.199 -> 0.2
- board text added: "SRAM IDT71V256SA 256kbit Mode LPC3 ALE1 EEPROM 24C02 - 2kbit TWID - addr 0x50 SDA - PD0 SCL - PD1 VCC - PD2 Voltage ref ADR380 2.048V 0.3% 25ppm/K VCC - PD3"
- board text removed: "SRAM IDT71V256SA 256kbit Mode LPC3 ALE1 EEPROM 24C02 - 2kbit TWID - addr 0x70 SDA - PD0 SCL - PD1 VCC - PD2 Voltage ref ADR380 2.048V 0.3% 25ppm/K VCC - PD3"

Commit message: Fix VBUS sense circuit
Voltage delivered with 2x(3k3) divider was too low, switch to 3x(3k3)
Connections:
- R23 pad 2: GND -> Net-(R23-Pad2)
- R23 pad 3: (no net) -> Net-(R23-Pad2)
- R23 pad 6: (no net) -> GND
Routing:
- net Net-(R23-Pad2): track 0.00 -> 0.80 mm

Commit message: Edit back silkscreen
Parts:
- added G***: LOGO, LOGO, B.Cu at (86.4, 14.0)
- added G***: LOGO, LOGO, B.Cu at (13.2, 13.8)
Other:
- board text added: "cpavlina/"
- board text added: "semianalog"

Commit message: Final PCB adjustment, DRC, and gerber rendering
Routing:
- net GND: track 546.0 -> 559.0 mm, vias 174 -> 184
- net /PA5: track 36.3 -> 38.9 mm
- net /PA6: track 37.9 -> 40.0 mm
- net /PA4: track 35.1 -> 37.3 mm
- net /PA7: track 39.5 -> 41.5 mm
- net /PA0: track 62.4 -> 64.1 mm
- net /PA3: track 34.8 -> 36.1 mm
- net /PA2: track 34.1 -> 35.0 mm
- net /PB0: track 50.9 -> 51.6 mm
